File: quad_copter_pcb/quad_copter_pcb.sch (KiCad schematic (older format))
At the start: 64 parts, among them J1 Conn_01x03_Male, J10 Conn_02x03_Odd_Even, J11 Conn_01x05, J12 USB_B_Micro, J2 Conn_01x03_Male, J3 Conn_01x03_Male, J4 Conn_01x03_Male, J5 Conn_02x05_Odd_Even, J6 Conn_02x02_Odd_Even, J7 Conn_01x05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

Commit message: Attempting to tune...
Parts:
- JP1: symbol SparkFun-Connectors:RJ11-6 -> quad_copter_pcb-rescue:RJ11-6-SparkFun-Connectors
- JP2: symbol SparkFun-RF:XBEE -> quad_copter_pcb-rescue:XBEE-SparkFun-RF
- S1, S2: symbol SparkFun-Switches:MOMENTARY-SWITCH-SPST-2-SMD-5.2MM -> quad_copter_pcb-rescue:MOMENTARY-SWITCH-SPST-2-SMD-5.2MM-SparkFun-Switches
- U3: symbol accel_gyro:accel_gyro_conn -> quad_copter_pcb-rescue:accel_gyro_conn-accel_gyro
- U4: symbol PIC32:PIC32MX775F512L-X_PT -> quad_copter_pcb-rescue:PIC32MX775F512L-X_PT-PIC32
Changed lines of the file:
@@
 EESchema Schematic File Version 4
 LIBS:quad_copter_pcb-cache
-EELAYER 26 0
+EELAYER 29 0
 EELAYER END
 $Descr C 22000 17000
@@
 $EndDescr
 $Comp
-L PIC32:PIC32MX775F512L-X_PT U4
+L quad_copter_pcb-rescue:PIC32MX775F512L-X_PT-PIC32 U4
 U 1 1 5BF9DBC4
 P 6650 5050
@@
 GND
 $Comp
-L SparkFun-RF:XBEE JP2
+L quad_copter_pcb-rescue:XBEE-SparkFun-RF JP2
 U 1 1 5BFB1552
 P 3850 12000
@@
 $EndComp
 $Comp
-L accel_gyro:accel_gyro_conn U3
+L quad_copter_pcb-rescue:accel_gyro_conn-accel_gyro U3
 U 1 1 5BFB1E23
 P 18900 12050
@@
 VDD3.3
 $Comp
-L SparkFun-Switches:MOMENTARY-SWITCH-SPST-2-SMD-5.2MM S1
+L quad_copter_pcb-rescue:MOMENTARY-SWITCH-SPST-2-SMD-5.2MM-SparkFun-Switches S1
 U 1 1 5BFBCCDC
 P 4600 3550
@@
 	5200 12100 5450 12100
 $Comp
-L SparkFun-Switches:MOMENTARY-SWITCH-SPST-2-SMD-5.2MM S2
+L quad_copter_pcb-rescue:MOMENTARY-SWITCH-SPST-2-SMD-5.2MM-SparkFun-Switches S2
 U 1 1 5BFDBEFA
 P 2550 9150
@@
 MCLR
 $Comp
-L SparkFun-Connectors:RJ11-6 JP1
+L quad_copter_pcb-rescue:RJ11-6-SparkFun-Connectors JP1
 U 1 1 5BFEB677
 P 5650 2000

Commit message: PCB updates
Parts:
- removed C14, C15: C15pF, Capacitor_SMD:C_0603_1608Metric_Pad1.05x0.95mm_HandSolder, symbol Device:C
- removed H1, H10, H2, H3, H4, H5, H6, H7, H8, H9: MountingHole_Pad, MountingHole:MountingHole_2.5mm_Pad, symbol Mechanical:MountingHole_Pad
- removed J7: Conn_01x05, Connector_PinHeader_2.54mm:PinHeader_1x05_P2.54mm_Vertical, symbol Connector_Generic:Conn_01x05
- removed J9: Conn_02x02_Odd_Even, Connector_PinHeader_2.54mm:PinHeader_2x02_P2.54mm_Vertical, symbol Connector_Generic:Conn_02x02_Odd_Even
- removed R6: R10k, Resistor_SMD:R_0805_2012Metric_Pad1.15x1.40mm_HandSolder, symbol Device:R
- removed R7: R470, Resistor_SMD:R_0603_1608Metric_Pad1.05x0.95mm_HandSolder, symbol Device:R
- removed S2: MOMENTARY-SWITCH-SPST-2-SMD-5.2MM, Switches:TACTILE_SWITCH_SMD_5.2MM, symbol quad_copter_pcb-rescue:MOMENTARY-SWITCH-SPST-2-SMD-5.2MM-SparkFun-Switches
- removed Y2: Crystal_GND23, Crystal:Crystal_SMD_7050-4Pin_7.0x5.0mm, symbol Device:Crystal_GND23
- added H15, H16: MountingHole, MountingHole:MountingHole_3.2mm_M3, symbol Mechanical:MountingHole
- renumbered H_4 to H14
Other:
- moved on the sheet: C4, C5, H11, H12, H13, H14, Y1
